File: KiCad Project/ledMatrixIT/ledMatrixIT.kicad_sch (KiCad schematic)
At the start: 156 parts, among them U1 IS31FL3731-QF, U2 XIAO-RP2040-DIP

Commit message: added schematic pdf to images directory and improved schematic readability
Other:
- title: (none) -> MatrixCard
Changed lines of the file:
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@@
 	(generator_version "8.0")
 	(paper "A4")
+	(title_block
+		(title "MatrixCard")
+		(date "2025-02-08")
+		(rev "1")
+	)
 	(junction
 		(at 88.9 35.56)
@@
 	)
 	(junction
+		(at 137.16 167.64)
+		(diameter 0)
+		(color 0 0 0 0)
+	)
+	(junction
 		(at 234.95 92.71)
 		(diameter 0)
@@
 	(wire
 		(pts
+			(xy 137.16 167.64) (xy 142.24 167.64)
+		)
+		(stroke
+			(width 0)
+			(type default)
+		)
+	)
+	(wire
+		(pts
 			(xy 116.84 97.79) (xy 111.76 102.87)
 		)
@@
 	(wire
 		(pts
-			(xy 124.46 160.02) (xy 127 160.02)
+			(xy 124.46 157.48) (xy 127 157.48)
 		)
 		(stroke
@@
 	(wire
 		(pts
-			(xy 87.63 147.32) (xy 91.44 147.32)
+			(xy 87.63 147.32) (xy 95.25 147.32)
 		)
 		(stroke
@@
 	(wire
 		(pts
-			(xy 127 160.02) (xy 127 162.56)
+			(xy 127 157.48) (xy 127 162.56)
 		)
 		(stroke
@@
 	(wire
 		(pts
-			(xy 135.89 167.64) (xy 142.24 167.64)
+			(xy 135.89 167.64) (xy 137.16 167.64)
 		)
 		(stroke
@@
 	(symbol
 		(lib_id "power:GND")
-		(at 124.46 160.02 0)
+		(at 124.46 157.48 0)
 		(unit 1)
 		(exclude_from_sim no)
@@
 		(dnp no)
 		(property "Reference" "#PWR012"
-			(at 124.46 166.37 0)
+			(at 124.46 163.83 0)
 			(effects
 				(font
@@
 		)
 		(property "Value" "GND"
-			(at 124.46 163.83 0)
+			(at 124.46 161.29 0)
 			(effects
 				(font
@@
 		)
 		(property "Footprint" ""
-			(at 124.46 160.02 0)
+			(at 124.46 157.48 0)
 			(effects
 				(font
@@
 		)
 		(property "Datasheet" ""
-			(at 124.46 160.02 0)
+			(at 124.46 157.48 0)
 			(effects
 				(font
@@
 		)
 		(property "Description" "Power symbol creates a global label with name \"GND\" , ground"
-			(at 124.46 160.02 0)
+			(at 124.46 157.48 0)
 			(effects
 				(font
@@
 		(dnp no)
 		(property "Reference" "C2"
-			(at 145.542 171.45 90)
+			(at 142.24 163.322 0)
 			(effects
 				(font
@@
 		)
 		(property "Value" "0.22uF"
-			(at 143.764 171.45 90)
+			(at 142.24 165.862 0)
 			(effects
 				(font
@@
 		(dnp no)
 		(property "Reference" "C3"
-			(at 142.748 171.45 90)
+			(at 148.59 161.544 0)
 			(effects
 				(font
@@
 		)
 		(property "Value" "0.22uF"
-			(at 145.288 171.45 90)
+			(at 148.59 164.084 0)
 			(effects
 				(font
@@
 	(symbol
 		(lib_id "power:GND")
-		(at 135.89 167.64 0)
+		(at 137.16 167.64 0)
 		(unit 1)
 		(exclude_from_sim no)
@@
 		(dnp no)
 		(property "Reference" "#PWR09"
-			(at 135.89 173.99 0)
+			(at 137.16 173.99 0)
 			(effects
 				(font
@@
 		)
 		(property "Value" "GND"
-			(at 135.89 171.45 0)
+			(at 137.16 171.45 0)
 			(effects
 				(font
@@
 		)
 		(property "Footprint" ""
-			(at 135.89 167.64 0)
+			(at 137.16 167.64 0)
 			(effects
 				(font
@@
 		)
 		(property "Datasheet" ""
-			(at 135.89 167.64 0)
+			(at 137.16 167.64 0)
 			(effects
 				(font
@@
 		)
 		(property "Description" "Power symbol creates a global label with name \"GND\" , ground"
-			(at 135.89 167.64 0)
+			(at 137.16 167.64 0)
 			(effects
 				(font
@@
 	(symbol
 		(lib_id "power:+3V0")
-		(at 91.44 147.32 0)
+		(at 95.25 147.32 0)
 		(unit 1)
 		(exclude_from_sim no)
@@
 		(dnp no)
 		(property "Reference" "#PWR05"
-			(at 91.44 151.13 0)
+			(at 95.25 151.13 0)
 			(effects
 				(font
@@
 		)
 		(property "Value" "+3V0"
-			(at 91.44 142.24 0)
+			(at 95.25 142.24 0)
 			(effects
 				(font
@@
 		)
 		(property "Footprint" ""
-			(at 91.44 147.32 0)
+			(at 95.25 147.32 0)
 			(effects
 				(font
@@
 		)
 		(property "Datasheet" ""
-			(at 91.44 147.32 0)
+			(at 95.25 147.32 0)
 			(effects
 				(font
@@
 		)
 		(property "Description" "Power symbol creates a global label with name \"+3V0\""
-			(at 91.44 147.32 0)
+			(at 95.25 147.32 0)
 			(effects
 				(font
